File: KiCad/PD_trigger_module.kicad_sch (KiCad schematic)
At the start: 22 parts, among them J1 Conn_01x01_Female, J2 Conn_01x01_Female, J3 Conn_01x01_Female, J4 Conn_01x01_Female, J5 USB_C_Receptacle_USB2.0, Q1 AON7403, U1 HUSB238

Commit message: Some minor corrections
Parts:
- J5: footprint _chips:USB_C_16pin -> _usb:TYPE_C_GCT_USB4505-03-0-A
Changed lines of the file:
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@@
   (symbol (lib_id "_chips:AON7403") (at 142.24 44.45 270) (mirror x) (unit 1)
     (in_bom yes) (on_board yes)
-    (property "Reference" "Q1" (id 0) (at 142.24 30.3743 90))
+    (property "Reference" "Q1" (id 0) (at 142.24 38.1 90))
     (property "Value" "AON7403" (id 1) (at 148.59 45.72 90))
     (property "Footprint" "_transistors:AON7403" (id 2) (at 144.78 39.37 0)
@@
   )
   (symbol (lib_id "Device:Fuse_Small") (at 102.87 45.72 0) (unit 1)
-    (in_bom yes) (on_board yes) (fields_autoplaced)
-    (property "Reference" "F1" (id 0) (at 102.87 41.3725 0))
-    (property "Value" "Fuse_Small" (id 1) (at 102.87 44.1476 0))
+    (in_bom yes) (on_board yes)
+    (property "Reference" "F1" (id 0) (at 102.87 43.18 0))
+    (property "Value" "Fuse_Small" (id 1) (at 102.87 44.1476 0)
+      (effects (font (size 1.27 1.27)) hide)
+    )
     (property "Footprint" "_chips:FuseHolder_1808" (id 2) (at 102.87 45.72 0)
       (effects (font (size 1.27 1.27)) hide)
@@
   (symbol (lib_id "Connector:USB_C_Receptacle_USB2.0") (at 74.93 60.96 0) (unit 1)
     (in_bom yes) (on_board yes)
-    (property "Reference" "J5" (id 0) (at 74.93 39.2135 0))
-    (property "Value" "USB_C_Receptacle_USB2.0" (id 1) (at 74.93 41.9886 0))
-    (property "Footprint" "_chips:USB_C_16pin" (id 2) (at 78.74 60.96 0)
+    (property "Reference" "J5" (id 0) (at 74.93 40.64 0))
+    (property "Value" "USB_C_Receptacle_USB2.0" (id 1) (at 74.93 41.9886 0)
+      (effects (font (size 1.27 1.27)) hide)
+    )
+    (property "Footprint" "_usb:TYPE_C_GCT_USB4505-03-0-A" (id 2) (at 78.74 60.96 0)
       (effects (font (size 1.27 1.27)) hide)
     )
@@
     )
     (path "/febe1f9a-ec1d-4b09-9aa9-b6db32363a29"
-      (reference "J5") (unit 1) (value "USB_C_Receptacle_USB2.0") (footprint "_chips:USB_C_16pin")
+      (reference "J5") (unit 1) (value "USB_C_Receptacle_USB2.0") (footprint "_usb:TYPE_C_GCT_USB4505-03-0-A")
     )
     (path "/14d47621-fb59-4b5a-87b0-d3f1d0ada326"
